File: electronics/RFID/RFID.kicad_pcb (KiCad board)
At the start: 2 copper layers, 20 parts, among them J1 USB_C_Receptacle_PowerOnly_6P, J2 Conn_01x10_Pin, J4 Conn_01x16_Pin, U1 AP63200WU, U2 74LVC2G14

Commit message: pcb
Parts:
- moved C2 28.8 mm to (124.2, 102.2), turned to 90 degrees
- moved U1 27.1 mm to (121.4, 102.4), turned to 90 degrees
- moved C3 23.2 mm to (117.7, 101.6), turned to -90 degrees
- moved C4 19.3 mm to (126.2, 95.1), turned to -90 degrees
- moved C5 15.7 mm to (124.2, 95.1), turned to -90 degrees
- moved C1 13.9 mm to (107.7, 59.8), turned to -90 degrees
- moved L1 9.30 mm to (119.9, 96.3), turned to 90 degrees
- moved R2 8.77 mm to (113.6, 105.3), turned to 180 degrees
- moved R3 3.79 mm to (113.6, 103.3), turned to 180 degrees
- moved J1 3.26 mm to (118.1, 111.2)
- moved JP1 3.26 mm to (109.8, 109.9)
Connections:
- C4 pad 1: /V3.3 -> +3.3V
- C5 pad 1: /V3.3 -> +3.3V
- L1 pad 2: /V3.3 -> +3.3V
- U1 pad 1: /V3.3 -> +3.3V
- U3 pad 2: unconnected-(U3-EN-Pad2) -> +3.3V
Routing:
- net +3.3V: track 0.00 -> 108.4 mm, vias 0 -> 5
- net +5V: track 10.1 -> 112.5 mm, vias 1 -> 0
- net Net-(J1-CC2): track 0.00 -> 6.67 mm
- net Net-(J1-CC1): track 0.00 -> 4.83 mm
- net Net-(U1-BST): track 0.00 -> 3.28 mm
- net Net-(U1-SW): track 0.00 -> 1.28 mm
- net GND: vias 1 -> 19
- added copper zone on F.Cu, net +3.3V
- added copper zone on F.Cu, net +5V
- added copper zone on B.Cu, net GND
- added copper zone on F.Cu, net GND
- added copper zone on F.Cu, net Net-(U1-SW)
Other:
- board outline added: 48.3 x 76.2 mm

Commit message: pcbV2
Parts:
- added J3: Conn Uart, Connector_PinHeader_2.54mm:PinHeader_1x04_P2.54mm_Vertical, F.Cu at (96.5, 94.0)
- added J5: Conn motion, Connector_PinHeader_2.54mm:PinHeader_1x04_P2.54mm_Vertical, F.Cu at (96.5, 68.2)
- J2: value Conn_01x10_Pin -> Conn deur; footprint Connector_PinSocket_2.54mm:PinSocket_1x10_P2.54mm_Vertical -> Connector_PinHeader_2.54mm:PinHeader_1x04_P2.54mm_Vertical
- RV1: moved to F.Cu
- moved RV1 58.4 mm to (136.1, 99.3), turned to 180 degrees
- moved J4 53.1 mm to (137.2, 94.5), turned to 0 degrees
- moved J2 46.3 mm to (96.5, 80.6), turned to 180 degrees
- moved U2 40.5 mm to (100.8, 68.5)
Connections:
- J2 pad 2: GND -> SensorDeur
- J2 pad 3: TX -> DeurControl
- J2 pad 4: RX -> +3.3V
- U2 pad 1: Net-(J2-Pin_8) -> Net-(J5-Pin_3)
- U2 pad 3: Net-(J2-Pin_7) -> Net-(J5-Pin_2)
- U3 pad 10: D1 -> SensorDeur
- U3 pad 11: D2 -> unconnected-(U3-27-Pad11)
- U3 pad 12: D3 -> RX
- U3 pad 13: D4 -> TX
- U3 pad 15: D5 -> unconnected-(U3-13-Pad15)
- U3 pad 16: D6 -> unconnected-(U3-D2-Pad16)
- U3 pad 17: D7 -> unconnected-(U3-D3-Pad17)
- U3 pad 21: unconnected-(U3-23-Pad21) -> D7
- U3 pad 22: unconnected-(U3-Pad22) -> D6
- U3 pad 23: TX -> D5
- U3 pad 24: RX -> D4
- U3 pad 25: SensorDeur -> D3
- U3 pad 27: DeurControl -> D2
- U3 pad 28: unconnected-(U3-18-Pad28) -> D1
- U3 pad 30: unconnected-(U3-17-Pad30) -> D0
- U3 pad 31: unconnected-(U3-16-Pad31) -> E
- U3 pad 32: unconnected-(U3-4-Pad32) -> RW
- U3 pad 33: M2 -> unconnected-(U3-0-Pad33)
- U3 pad 34: M1 -> RS
- U3 pad 6: RS -> unconnected-(U3-35-Pad6)
- U3 pad 7: RW -> M1
- U3 pad 8: E -> M2
- U3 pad 9: D0 -> DeurControl
Routing:
- net +5V: track 112.5 -> 136.8 mm, vias 0 -> 1
- net Net-(J2-Pin_7): track 14.3 -> 0.00 mm
- net Net-(J2-Pin_8): track 12.0 -> 0.00 mm
- net Net-(J5-Pin_3): track 0.00 -> 8.76 mm
- net M1: track 9.73 -> 2.97 mm
- net +3.3V: track 108.4 -> 102.7 mm
- net Net-(J5-Pin_2): track 0.00 -> 4.54 mm
- net Net-(J4-Pin_3): track 14.6 -> 10.2 mm
- net TX: track 7.61 -> 10.9 mm
- net RX: track 7.61 -> 10.9 mm
- net GND: track 2.04 -> 3.61 mm, vias 19 -> 25
- net E: track 8.58 -> 7.24 mm
- net D0: track 8.58 -> 7.24 mm
- net RW: track 8.58 -> 7.24 mm
- net DeurControl: track 7.45 -> 8.58 mm
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Other:
- board text removed: "footprint van lcd nog is nachecken"
- board text removed: "hercheck ook footprint trimmer RV1"
- board text removed: "let op bounding box van lcd (zeer groot en niet getoond)"

Commit message: pcbV2
Parts:
- moved H1 4.31 mm to (98.0, 48.3)
- moved H2 3.30 mm to (136.1, 48.3)
- moved H4 2.92 mm to (98.0, 107.3)
- moved H3 0.97 mm to (136.1, 107.7)
Routing:
- net GND: vias 25 -> 30
Other:
- board size 48.3 x 76.2 mm -> 48.3 x 71.1 mm
- board text added: "Groep 8 RFID"
Changed lines of the file:
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@@
   )
   (footprint "MountingHole:MountingHole_4mm" (layer "F.Cu")
-    (at 100.965 107.315)
+    (at 98.044 107.315)
     (descr "Mounting Hole 4mm, no annular")
     (tags "mounting hole 4mm no annular")
@@
   )
   (footprint "MountingHole:MountingHole_4mm" (layer "F.Cu")
-    (at 135.255 107.315)
+    (at 136.144 107.696)
     (descr "Mounting Hole 4mm, no annular")
     (tags "mounting hole 4mm no annular")
@@
     (property "ki_keywords" "mounting hole")
     (attr exclude_from_pos_files)
-    (fp_text reference "H3" (at -4.826 3.937) (layer "F.SilkS")
+    (fp_text reference "H3" (at -5.207 2.413) (layer "F.SilkS")
         (effects (font (size 1 1) (thickness 0.15)))
     )
@@
   )
   (footprint "MountingHole:MountingHole_4mm" (layer "F.Cu")
-    (at 135.255 45.085)
+    (at 136.144 48.26)
     (descr "Mounting Hole 4mm, no annular")
     (tags "mounting hole 4mm no annular")
@@
     (property "ki_keywords" "mounting hole")
     (attr exclude_from_pos_files)
-    (fp_text reference "H2" (at 0 -5) (layer "F.SilkS")
+    (fp_text reference "H2" (at -4.572 -3.556) (layer "F.SilkS")
         (effects (font (size 1 1) (thickness 0.15)))
     )
@@
   )
   (footprint "MountingHole:MountingHole_4mm" (layer "F.Cu")
-    (at 100.965 45.085)
+    (at 98.044 48.26)
     (descr "Mounting Hole 4mm, no annular")
     (tags "mounting hole 4mm no annular")
@@
     (property "ki_keywords" "mounting hole")
     (attr exclude_from_pos_files)
-    (fp_text reference "H1" (at 0 -5) (layer "F.SilkS")
+    (fp_text reference "H1" (at 5.08 -3.048) (layer "F.SilkS")
         (effects (font (size 1 1) (thickness 0.15)))
     )
@@
         (effects (font (size 1 1) (thickness 0.15)))
     )
-    (fp_text user "${REFERENCE}" (at 0 0) (layer "F.Fab")
+    (fp_text user "${REFERENCE}" (at -3.937 4.318) (layer "F.Fab")
         (effects (font (size 1 1) (thickness 0.15)))
     )
@@
     )
   )
-  (gr_rect (start 92.71 38.1) (end 140.97 114.3)
+  (gr_rect (start 92.71 43.18) (end 140.97 114.3)
     (stroke (width 0.1) (type default)) (fill none) (layer "Edge.Cuts"))
+  (gr_text "Groep 8 RFID" (at 126.365 113.411) (layer "F.SilkS")
+    (effects (font (size 1 1) (thickness 0.15)) (justify left bottom))
+  )
   (segment (start 104.7434 54.3924) (end 104.7434 56.9324) (width 0.5) (layer "F.Cu") (net 1))
   (segment (start 98.298 86.36) (end 96.52 86.36) (width 0.5) (layer "F.Cu") (net 1))
@@
   (via (at 115.443 109.855) (size 0.8) (drill 0.4) (layers "F.Cu" "B.Cu") (free) (net 2))
   (via (at 107.188 87.376) (size 0.8) (drill 0.4) (layers "F.Cu" "B.Cu") (free) (net 2))
+  (via (at 102.5906 104.1908) (size 0.8) (drill 0.4) (layers "F.Cu" "B.Cu") (free) (net 2))
   (via (at 121.031 110.109) (size 0.8) (drill 0.4) (layers "F.Cu" "B.Cu") (free) (net 2))
   (via (at 98.425 68.326) (size 0.8) (drill 0.4) (layers "F.Cu" "B.Cu") (free) (net 2))
@@
   (via (at 107.188 67.183) (size 0.8) (drill 0.4) (layers "F.Cu" "B.Cu") (free) (net 2))
   (via (at 139.192 100.711) (size 0.8) (drill 0.4) (layers "F.Cu" "B.Cu") (free) (net 2))
+  (via (at 102.4128 60.6552) (size 0.8) (drill 0.4) (layers "F.Cu" "B.Cu") (free) (net 2))
   (via (at 107.442 55.372) (size 0.8) (drill 0.4) (layers "F.Cu" "B.Cu") (free) (net 2))
   (via (at 126.492 101.473) (size 0.8) (drill 0.4) (layers "F.Cu" "B.Cu") (free) (net 2))
   (via (at 133.731 95.885) (size 0.8) (drill 0.4) (layers "F.Cu" "B.Cu") (free) (net 2))
   (via (at 99.187 64.389) (size 0.8) (drill 0.4) (layers "F.Cu" "B.Cu") (free) (net 2))
+  (via (at 96.5708 101.1428) (size 0.8) (drill 0.4) (layers "F.Cu" "B.Cu") (free) (net 2))
   (via (at 123.952 99.822) (size 0.8) (drill 0.4) (layers "F.Cu" "B.Cu") (free) (net 2))
   (via (at 110.998 104.14) (size 0.8) (drill 0.4) (layers "F.Cu" "B.Cu") (free) (net 2))
@@
   (via (at 126.492 97.663) (size 0.8) (drill 0.4) (layers "F.Cu" "B.Cu") (free) (net 2))
   (via (at 121.539 106.299) (size 0.8) (drill 0.4) (layers "F.Cu" "B.Cu") (free) (net 2))
+  (via (at 99.441 60.7822) (size 0.8) (drill 0.4) (layers "F.Cu" "B.Cu") (free) (net 2))
+  (via (at 102.4382 80.4926) (size 0.8) (drill 0.4) (layers "F.Cu" "B.Cu") (free) (net 2))
   (segment (start 115.697 106.68) (end 116.545 107.528) (width 0.5) (layer "F.Cu") (net 3))
   (segment (start 116.79 109.22) (end 119.34 109.22) (width 0.5) (layer "F.Cu") (net 3))
@@
     (polygon
       (pts
-        (xy 92.71 38.1)
-        (xy 140.97 38.1)
+        (xy 92.71 43.18)
+        (xy 140.97 43.18)
         (xy 140.97 114.3)
         (xy 92.71 114.3)
@@
     (polygon
       (pts
-        (xy 105.283 37.973)
+        (xy 105.283 43.053)
         (xy 105.283 52.451)
         (xy 130.429 52.451)
-        (xy 130.429 37.973)
+        (xy 130.429 43.053)
       )
     )
@@
     (polygon
       (pts
-        (xy 92.71 38.1)
-        (xy 140.97 38.1)
+        (xy 92.71 43.18)
+        (xy 140.97 43.18)
         (xy 140.97 114.3)
         (xy 92.71 114.3)

Commit message: PCBV3
Routing:
- net GND: vias 30 -> 107

Commit message: pcbVfinal?
Parts:
- J3: footprint Connector_PinHeader_2.54mm:PinHeader_1x04_P2.54mm_Vertical -> Connector_PinHeader_2.00mm:PinHeader_1x04_P2.00mm_Vertical
- U1: value AP63200WU -> AP63202WU
- moved J3 1.38 mm to (96.5, 92.6)
Connections:
- J3 pad 2: TX -> +5V
- J3 pad 3: RX -> TX
- J3 pad 4: +3.3V -> RX
Routing:
- net +3.3V: track 102.7 -> 86.5 mm, vias 5 -> 4
- net +5V: track 136.8 -> 141.2 mm
- net TX: track 10.9 -> 9.77 mm
- net RX: track 10.9 -> 9.99 mm
Other:
- board text added: "HY2.0 spacing"

Commit message: proxima fixed :chad:
fixed by proxi hihihiih love you <3
Parts:
- L1: footprint Inductor_SMD:L_Bourns-SRN6028 -> KiCad:SRR4828A3R9Y
- moved L1 0.20 mm to (119.7, 96.3), turned to 180 degrees
Routing:
- net Net-(U1-SW): track 1.28 -> 5.21 mm
- net +3.3V: track 86.5 -> 88.5 mm
Changed lines of the file:
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@@
   (net 43 "unconnected-(U3-D3-Pad17)")
   (net 44 "unconnected-(U3-0-Pad33)")
-  (footprint "Inductor_SMD:L_Bourns-SRN6028" (layer "F.Cu")
-    (at 119.888 96.266 90)
-    (descr "Bourns SRN6028 series SMD inductor")
-    (tags "Bourns SRN6028 SMD inductor")
+  (footprint "KiCad:SRR4828A3R9Y" (layer "F.Cu")
+    (at 119.689398 96.277231 180)
+    (descr "SRR4828A-3R9Y-2")
+    (tags "Inductor")
     (property "Sheetfile" "RFID.kicad_sch")
     (property "Sheetname" "")
@@
     (property "ki_keywords" "inductor choke coil reactor magnetic")
     (attr smd)
-    (fp_text reference "L1" (at 0 0 90) (layer "F.SilkS")
-        (effects (font (size 1 1) (thickness 0.15)))
-    )
-    (fp_text value "3.9µH" (at 0 -4 90) (layer "F.Fab")
-        (effects (font (size 1 1) (thickness 0.15)))
-    )
-    (fp_text user "${REFERENCE}" (at 0 0 90) (layer "F.Fab")
-        (effects (font (size 1 1) (thickness 0.15)))
-    )
-    (fp_line (start -3.4 -3.2) (end -3.4 -2)
-      (stroke (width 0.12) (type solid)) (layer "F.SilkS"))
-    (fp_line (start -3.4 -3.2) (end -2 -3.2)
-      (stroke (width 0.12) (type solid)) (layer "F.SilkS"))
-    (fp_line (start -3.4 3.2) (end -3.4 2)
-      (stroke (width 0.12) (type solid)) (layer "F.SilkS"))
-    (fp_line (start -3.4 3.2) (end -2 3.2)
-      (stroke (width 0.12) (type solid)) (layer "F.SilkS"))
-    (fp_line (start 3.4 -3.2) (end 2 -3.2)
-      (stroke (width 0.12) (type solid)) (layer "F.SilkS"))
-    (fp_line (start 3.4 -3.2) (end 3.4 -2)
-      (stroke (width 0.12) (type solid)) (layer "F.SilkS"))
-    (fp_line (start 3.4 3.2) (end 2 3.2)
-      (stroke (width 0.12) (type solid)) (layer "F.SilkS"))
-    (fp_line (start 3.4 3.2) (end 3.4 2)
-      (stroke (width 0.12) (type solid)) (layer "F.SilkS"))
-    (fp_line (start -3.3 -3.1) (end -3.3 3.1)
-      (stroke (width 0.05) (type solid)) (layer "F.CrtYd"))
-    (fp_line (start -3.3 -3.1) (end 3.3 -3.1)
-      (stroke (width 0.05) (type solid)) (layer "F.CrtYd"))
-    (fp_line (start 3.3 -3.1) (end 3.3 3.1)
-      (stroke (width 0.05) (type solid)) (layer "F.CrtYd"))
-    (fp_line (start 3.3 3.1) (end -3.3 3.1)
-      (stroke (width 0.05) (type solid)) (layer "F.CrtYd"))
-    (fp_line (start -3.3 -3.1) (end -3.3 3.1)
-      (stroke (width 0.1) (type solid)) (layer "F.Fab"))
-    (fp_line (start -3.3 -3.1) (end 3.3 -3.1)
-      (stroke (width 0.1) (type solid)) (layer "F.Fab"))
-    (fp_line (start 3.3 -3.1) (end 3.3 3.1)
-      (stroke (width 0.1) (type solid)) (layer "F.Fab"))
-    (fp_line (start 3.3 3.1) (end -3.3 3.1)
-      (stroke (width 0.1) (type solid)) (layer "F.Fab"))
-    (pad "1" smd rect (at -2.35 0 90) (size 1.6 5.7) (layers "F.Cu" "F.Paste" "F.Mask")
+    (fp_text reference "L1" (at 0 0) (layer "F.SilkS")
+        (effects (font (size 1.27 1.27) (thickness 0.254)))
+    )
+    (fp_text value "3.9µH" (at 0 0) (layer "F.SilkS") hide
+        (effects (font (size 1.27 1.27) (thickness 0.254)))
+    )
+    (fp_text user "${REFERENCE}" (at 0 0) (layer "F.Fab")
+        (effects (font (size 1.27 1.27) (thickness 0.254)))
+    )
+    (fp_line (start -2.4 -2.4) (end -2.4 2.4)
+      (stroke (width 0.1) (type solid)) (layer "F.SilkS"))
+    (fp_line (start 2.4 -2.4) (end 2.4 2.4)
+      (stroke (width 0.1) (type solid)) (layer "F.SilkS"))
+    (fp_line (start -3.4 -3.565) (end 3.4 -3.565)
+      (stroke (width 0.1) (type solid)) (layer "F.CrtYd"))
+    (fp_line (start -3.4 3.565) (end -3.4 -3.565)
+      (stroke (width 0.1) (type solid)) (layer "F.CrtYd"))
+    (fp_line (start 3.4 -3.565) (end 3.4 3.565)
+      (stroke (width 0.1) (type solid)) (layer "F.CrtYd"))
+    (fp_line (start 3.4 3.565) (end -3.4 3.565)
+      (stroke (width 0.1) (type solid)) (layer "F.CrtYd"))
+    (fp_line (start -2.4 -2.4) (end 2.4 -2.4)
+      (stroke (width 0.2) (type solid)) (layer "F.Fab"))
+    (fp_line (start -2.4 2.4) (end -2.4 -2.4)
+      (stroke (width 0.2) (type solid)) (layer "F.Fab"))
+    (fp_line (start 2.4 -2.4) (end 2.4 2.4)
+      (stroke (width 0.2) (type solid)) (layer "F.Fab"))
+    (fp_line (start 2.4 2.4) (end -2.4 2.4)
+      (stroke (width 0.2) (type solid)) (layer "F.Fab"))
+    (pad "1" smd rect (at 0 -1.575 270) (size 1.98 4.2) (layers "F.Cu" "F.Paste" "F.Mask")
       (net 4 "Net-(U1-SW)") (pinfunction "1") (pintype "passive"))
-    (pad "2" smd rect (at 2.35 0 90) (size 1.6 5.7) (layers "F.Cu" "F.Paste" "F.Mask")
+    (pad "2" smd rect (at 0 1.575 270) (size 1.98 4.2) (layers "F.Cu" "F.Paste" "F.Mask")
       (net 1 "+3.3V") (pinfunction "2") (pintype "passive"))
-    (model "${KICAD6_3DMODEL_DIR}/Inductor_SMD.3dshapes/L_Bourns-SRN6028.wrl"
+    (model "SRR4828A-3R9Y.stp"
       (offset (xyz 0 0 0))
       (scale (xyz 1 1 1))
@@
   )
   (segment (start 104.7434 54.3924) (end 104.7434 56.9324) (width 0.5) (layer "F.Cu") (net 1))
+  (segment (start 119.689398 70.860398) (end 119.689398 94.702231) (width 0.5) (layer "F.Cu") (net 1))
   (segment (start 100.838 73.025) (end 96.52 73.025) (width 0.5) (layer "F.Cu") (net 1))
-  (segment (start 115.951 95.631) (end 117.666 93.916) (width 0.5) (layer "F.Cu") (net 1))
-  (segment (start 119.888 71.059) (end 119.888 93.916) (width 0.5) (layer "F.Cu") (net 1))
-  (segment (start 105.7614 56.9324) (end 107.696 58.867) (width 0.5) (layer "F.Cu") (net 1))
-  (segment (start 117.666 93.916) (end 119.888 93.916) (width 0.5) (layer "F.Cu") (net 1))
-  (segment (start 107.696 58.867) (end 119.888 71.059) (width 0.5) (layer "F.Cu") (net 1))
+  (segment (start 117.768769 94.702231) (end 115.951 96.52) (width 0.5) (layer "F.Cu") (net 1))
   (segment (start 120.462 103.4995) (end 119.5125 103.4995) (width 0.5) (layer "F.Cu") (net 1))
+  (segment (start 119.666648 94.430447) (end 118.556648 94.430447) (width 0.5) (layer "F.Cu") (net 1))
+  (segment (start 119.689398 94.702231) (end 119.587029 94.8046) (width 0.5) (layer "F.Cu") (net 1))
+  (segment (start 115.951 96.52) (end 115.951 97.79) (width 0.5) (layer "F.Cu") (net 1))
+  (segment (start 106.9645 58.1355) (end 119.689398 70.860398) (width 0.5) (layer "F.Cu") (net 1))
+  (segment (start 105.7614 56.9324) (end 106.9645 58.1355) (width 0.5) (layer "F.Cu") (net 1))
   (segment (start 119.5125 103.4995) (end 119.507 103.505) (width 0.5) (layer "F.Cu") (net 1))
-  (segment (start 115.951 97.79) (end 115.951 95.631) (width 0.5) (layer "F.Cu") (net 1))
+  (segment (start 119.689398 94.702231) (end 117.768769 94.702231) (width 0.5) (layer "F.Cu") (net 1))
+  (segment (start 106.9645 58.1355) (end 107.696 58.867) (width 0.5) (layer "F.Cu") (net 1))
   (segment (start 104.7434 56.9324) (end 105.7614 56.9324) (width 0.5) (layer "F.Cu") (net 1))
   (segment (start 100.838 69.5905) (end 100.838 71.12) (width 0.5) (layer "F.Cu") (net 1))
@@
   (segment (start 132.715 101.092) (end 132.715 94.996) (width 0.5) (layer "B.Cu") (net 3))
   (segment (start 133.6675 94.0435) (end 135.763 91.948) (width 0.5) (layer "B.Cu") (net 3))
+  (segment (start 119.666648 98.773352) (end 119.38 99.06) (width 0.25) (layer "F.Cu") (net 4))
   (segment (start 121.412 101.2245) (end 121.412 99.949) (width 0.5) (layer "F.Cu") (net 4))
+  (segment (start 119.666648 97.580447) (end 119.666648 98.773352) (width 0.25) (layer "F.Cu") (net 4))
+  (segment (start 119.38 98.999) (end 117.729 100.65) (width 0.25) (layer "F.Cu") (net 4))
   (segment (start 118.303 102.55) (end 119.6285 101.2245) (width 0.5) (layer "F.Cu") (net 5))
   (segment (start 119.6285 101.2245) (end 120.462 101.2245) (width 0.5) (layer "F.Cu") (net 5))
